Commit message: workable teleop

File: config/humanoid_arm.urdf (robot description, URDF)
Before this commit: robot humand_arm, 5 links, 4 joints
Links:
- removed link elbow
- removed link fix1
- removed link hand
- removed link shoulder_z
- removed link wrist_y
- added link ${name}/elbow; visual cylinder length=0.20 radius=0.05
- added link ${name}/fix1; visual cylinder length=0.1 radius=0.05
- added link ${name}/hand; visual sphere radius=0.06
- added link ${name}/shoulder_z; visual cylinder length=0.20 radius=0.05
- added link ${name}/wrist_x; visual cylinder length=0.07 radius=0.05
Joints:
- removed joint elbow_wrist
- removed joint fix1_shoulder
- removed joint shoulder_elbow
- removed joint wrist_hand
- added joint ${name}/elbow_wrist: type fixed, parent ${name}/elbow, child ${name}/wrist_x, origin xyz=0 0 0.2 rpy=0 0 0
- added joint ${name}/fix1_shoulder: type fixed, parent ${name}/fix1, child ${name}/shoulder_z, origin xyz=0 0 0.0 rpy=0 0 0
- added joint ${name}/shoulder_elbow: type fixed, parent ${name}/shoulder_z, child ${name}/elbow, origin xyz=0 0 0.2 rpy=0 0 0
- added joint ${name}/wrist_hand: type fixed, parent ${name}/wrist_x, child ${name}/hand, origin xyz=0 0 0.07 rpy=0 0 0
